Commit message: added the new model adjusted the urdf files need to fix the sensor origins

File: workspace/jig_description/urdf/Main_jig.urdf.xacro (robot description, xacro)
@@ -4,4 +4,5 @@
   <xacro:include filename="$(find jig_description)/urdf/base.urdf.xacro"/>
   <xacro:include filename="$(find jig_description)/urdf/lidar.urdf.xacro"/>
+  <xacro:include filename="$(find jig_description)/urdf/realsense.urdf.xacro"/>
   <xacro:include filename="$(find jig_description)/urdf/gazebo_components.urdf.xacro"/>
 </robot>

File: workspace/jig_description/urdf/base.urdf.xacro (robot description, xacro)
@@ -8,5 +8,5 @@
       <origin xyz="0 0 0" rpy="0 0 0"/>
       <geometry>
-        <mesh filename="package://jig_description/meshes/jig_base.stl"
+        <mesh filename="package://jig_description/meshes/jig_base_v2.stl"
               scale="0.001 0.001 0.001"/>
       </geometry>
@@ -18,5 +18,5 @@
       <origin xyz="0 0 0" rpy="0 0 0"/>
       <geometry>
-        <mesh filename="package://jig_description/meshes/jig_base.stl"
+        <mesh filename="package://jig_description/meshes/jig_base_v2.stl"
               scale="0.001 0.001 0.001"/>
       </geometry>

File: workspace/jig_description/urdf/realsense.urdf.xacro (robot description, xacro)
@@ -2,16 +2,16 @@
 <robot xmlns:xacro="http://www.ros.org/wiki/xacro">
   <!-- ═══════════════════════════════════════════════════════════
-       LIDAR PARAMETERS
+       REALSENSE PARAMETERS
   ═══════════════════════════════════════════════════════════ -->
-  <xacro:property name="lidar_xyz"         value="0.025 -0.005 0.035"/>
-  <xacro:property name="lidar_rpy"         value="0 1.57 0"/>
+  <xacro:property name="lidar_xyz"         value="0.050 -0.001 -0.01"/>
+  <xacro:property name="lidar_rpy"         value="0 0 0"/>
   <!-- ═══════════════════════════════════════════════════════════
-       LIDAR LINK (MID360 with built-in IMU)
+       REALSENSE LINK
   ═══════════════════════════════════════════════════════════ -->
-  <link name="lidar_link">
+  <link name="camera_link">
     <visual>
       <origin xyz="0 0 0" rpy="0 0 0"/>
       <geometry>
-        <mesh filename="package://jig_description/meshes/mid360.stl"
+        <mesh filename="package://jig_description/meshes/realsense.stl"
               scale="0.001 0.001 0.001"/>
       </geometry>
@@ -23,5 +23,5 @@
       <origin xyz="0 0 0" rpy="0 0 0"/>
       <geometry>
-        <mesh filename="package://jig_description/meshes/mid360.stl"
+        <mesh filename="package://jig_description/meshes/realsense.stl"
               scale="0.001 0.001 0.001"/>
       </geometry>
@@ -35,9 +35,9 @@
   </link>
   <!-- ═══════════════════════════════════════════════════════════
-       LIDAR JOINT
+       REALSENSE JOINT
   ═══════════════════════════════════════════════════════════ -->
-  <joint name="base_to_lidar" type="fixed">
+  <joint name="base_to_camera" type="fixed">
     <parent link="base_link"/>
-    <child link="lidar_link"/>
+    <child link="camera_link"/>
     <origin xyz="${lidar_xyz}" rpy="${lidar_rpy}"/>
   </joint>
