Commit message: added realsense plugin

File: workspace/jig_description/urdf/gazebo_components.urdf.xacro (robot description, xacro)
@@ -27,5 +27,4 @@
             <samples>420</samples>
             <resolution>1</resolution>
-            <resolution>0.1047</resolution>
             <min_angle>-3.1415</min_angle>
             <max_angle>3.1415</max_angle>
@@ -34,5 +33,4 @@
             <samples>40</samples>
             <resolution>1</resolution>
-            <resolution>0.1047</resolution>
             <min_angle>0</min_angle>
             <max_angle>0.6109</max_angle>
@@ -117,3 +115,57 @@
     </sensor>
   </gazebo>
+  <!-- ═══════════════════════════════════════════════════════════
+       REALSENSE D435 — RGB CAMERA
+  ═══════════════════════════════════════════════════════════ -->
+  <gazebo reference="camera_link">
+    <sensor name="rgb_camera" type="camera">
+      <always_on>true</always_on>
+      <update_rate>30</update_rate>
+      <topic>/camera/color/image_raw</topic>
+      <visualize>true</visualize>
+      <camera>
+        <horizontal_fov>1.2112</horizontal_fov>
+        <image>
+          <width>1280</width>
+          <height>720</height>
+          <format>R8G8B8</format>
+        </image>
+        <clip>
+          <near>0.1</near>
+          <far>100</far>
+        </clip>
+        <noise>
+          <type>gaussian</type>
+          <mean>0.0</mean>
+          <stddev>0.007</stddev>
+        </noise>
+      </camera>
+    </sensor>
+    <!-- ═══════════════════════════════════════════════════════
+         REALSENSE D435 — DEPTH CAMERA
+    ═══════════════════════════════════════════════════════ -->
+    <sensor name="depth_camera" type="depth_camera">
+      <always_on>true</always_on>
+      <update_rate>30</update_rate>
+      <topic>/camera/depth/image_rect_raw</topic>
+      <visualize>true</visualize>
+      <camera>
+        <horizontal_fov>1.4835</horizontal_fov>
+        <image>
+          <width>1280</width>
+          <height>720</height>
+          <format>R_FLOAT32</format>
+        </image>
+        <clip>
+          <near>0.1</near>
+          <far>10.0</far>
+        </clip>
+        <noise>
+          <type>gaussian</type>
+          <mean>0.0</mean>
+          <stddev>0.01</stddev>
+        </noise>
+      </camera>
+    </sensor>
+  </gazebo>
 </robot>

File: workspace/jig_description/urdf/realsense.urdf.xacro (robot description, xacro)
@@ -2,8 +2,8 @@
 <robot xmlns:xacro="http://www.ros.org/wiki/xacro">
   <!-- ═══════════════════════════════════════════════════════════
-       REALSENSE PARAMETERS
+       REALSENSE D435 PARAMETERS
   ═══════════════════════════════════════════════════════════ -->
-  <xacro:property name="lidar_xyz"         value="0.050 -0.001 -0.01"/>
-  <xacro:property name="lidar_rpy"         value="0 0 0"/>
+  <xacro:property name="camera_xyz" value="0.050 -0.001 -0.01"/>
+  <xacro:property name="camera_rpy" value="0 0 0"/>
   <!-- ═══════════════════════════════════════════════════════════
        REALSENSE LINK
@@ -16,6 +16,6 @@
               scale="0.001 0.001 0.001"/>
       </geometry>
-      <material name="red">
-        <color rgba="0.8 0.0 0.0 1.0"/>
+      <material name="silver">
+        <color rgba="0.7 0.7 0.7 1.0"/>
       </material>
     </visual>
@@ -29,16 +29,23 @@
     <inertial>
       <origin xyz="0 0 0" rpy="0 0 0"/>
-      <mass value="0.3"/>
+      <mass value="0.072"/>
       <inertia ixx="0.001" ixy="0" ixz="0"
                iyy="0.001" iyz="0" izz="0.001"/>
     </inertial>
   </link>
+  <!-- Optical frame for ROS convention (Z forward, X right, Y down) -->
+  <link name="camera_optical_link"/>
   <!-- ═══════════════════════════════════════════════════════════
-       REALSENSE JOINT
+       REALSENSE JOINTS
   ═══════════════════════════════════════════════════════════ -->
   <joint name="base_to_camera" type="fixed">
     <parent link="base_link"/>
     <child link="camera_link"/>
-    <origin xyz="${lidar_xyz}" rpy="${lidar_rpy}"/>
+    <origin xyz="${camera_xyz}" rpy="${camera_rpy}"/>
+  </joint>
+  <joint name="camera_optical_joint" type="fixed">
+    <parent link="camera_link"/>
+    <child link="camera_optical_link"/>
+    <origin xyz="0 0 0" rpy="-1.5707 0 -1.5707"/>
   </joint>
 </robot>

Commit message: fixed the real sense sim error updated the docker files

File: workspace/jig_description/urdf/gazebo_components.urdf.xacro (robot description, xacro)
@@ -115,8 +115,8 @@
     </sensor>
   </gazebo>
-  <!-- ═══════════════════════════════════════════════════════════
+   <!-- ═══════════════════════════════════════════════════════════
        REALSENSE D435 — RGB CAMERA
   ═══════════════════════════════════════════════════════════ -->
-  <gazebo reference="camera_link">
+  <gazebo reference="camera_color_frame">
     <sensor name="rgb_camera" type="camera">
       <always_on>true</always_on>
@@ -127,6 +127,6 @@
         <horizontal_fov>1.2112</horizontal_fov>
         <image>
-          <width>1280</width>
-          <height>720</height>
+          <width>640</width>
+          <height>480</height>
           <format>R8G8B8</format>
         </image>
@@ -142,7 +142,9 @@
       </camera>
     </sensor>
-    <!-- ═══════════════════════════════════════════════════════
-         REALSENSE D435 — DEPTH CAMERA
-    ═══════════════════════════════════════════════════════ -->
+  </gazebo>
+  <!-- ═══════════════════════════════════════════════════════════
+       REALSENSE D435 — DEPTH CAMERA
+  ═══════════════════════════════════════════════════════════ -->
+  <gazebo reference="camera_depth_frame">
     <sensor name="depth_camera" type="depth_camera">
       <always_on>true</always_on>
@@ -153,6 +155,6 @@
         <horizontal_fov>1.4835</horizontal_fov>
         <image>
-          <width>1280</width>
-          <height>720</height>
+          <width>640</width>
+          <height>480</height>
           <format>R_FLOAT32</format>
         </image>
@@ -169,3 +171,3 @@
     </sensor>
   </gazebo>
-</robot>
+  </robot>

File: workspace/jig_description/urdf/realsense.urdf.xacro (robot description, xacro)
@@ -4,25 +4,21 @@
        REALSENSE D435 PARAMETERS
   ═══════════════════════════════════════════════════════════ -->
-  <xacro:property name="camera_xyz" value="0.050 -0.001 -0.01"/>
+  <xacro:property name="camera_xyz" value="0.065 -0.015 -0.01"/>
   <xacro:property name="camera_rpy" value="0 0 0"/>
   <!-- ═══════════════════════════════════════════════════════════
-       REALSENSE LINK
+       REALSENSE LINKS
   ═══════════════════════════════════════════════════════════ -->
+  <link name="camera_bottom_screw_frame"/>
   <link name="camera_link">
     <visual>
-      <origin xyz="0 0 0" rpy="0 0 0"/>
+      <origin xyz="0 0 0" rpy="-1.57 0 -1.57"/>
       <geometry>
-        <mesh filename="package://jig_description/meshes/realsense.stl"
-              scale="0.001 0.001 0.001"/>
+        <mesh filename="file://$(find realsense2_description)/meshes/d435.dae"/>
       </geometry>
-      <material name="silver">
-        <color rgba="0.7 0.7 0.7 1.0"/>
-      </material>
     </visual>
     <collision>
       <origin xyz="0 0 0" rpy="0 0 0"/>
       <geometry>
-        <mesh filename="package://jig_description/meshes/realsense.stl"
-              scale="0.001 0.001 0.001"/>
+        <box size="0.025 0.090 0.025"/>
       </geometry>
     </collision>
@@ -34,6 +30,8 @@
     </inertial>
   </link>
-  <!-- Optical frame for ROS convention (Z forward, X right, Y down) -->
-  <link name="camera_optical_link"/>
+  <link name="camera_depth_frame"/>
+  <link name="camera_depth_optical_frame"/>
+  <link name="camera_color_frame"/>
+  <link name="camera_color_optical_frame"/>
   <!-- ═══════════════════════════════════════════════════════════
        REALSENSE JOINTS
@@ -41,10 +39,30 @@
   <joint name="base_to_camera" type="fixed">
     <parent link="base_link"/>
-    <child link="camera_link"/>
+    <child link="camera_bottom_screw_frame"/>
     <origin xyz="${camera_xyz}" rpy="${camera_rpy}"/>
   </joint>
-  <joint name="camera_optical_joint" type="fixed">
+  <joint name="camera_link_joint" type="fixed">
+    <parent link="camera_bottom_screw_frame"/>
+    <child link="camera_link"/>
+    <origin xyz="0 0.0175 0.0125" rpy="0 0 0"/>
+  </joint>
+  <joint name="camera_depth_joint" type="fixed">
     <parent link="camera_link"/>
-    <child link="camera_optical_link"/>
+    <child link="camera_depth_frame"/>
+    <origin xyz="0 0 0" rpy="0 0 0"/>
+  </joint>
+  <joint name="camera_depth_optical_joint" type="fixed">
+    <parent link="camera_depth_frame"/>
+    <child link="camera_depth_optical_frame"/>
+    <origin xyz="0 0 0" rpy="-1.5707 0 -1.5707"/>
+  </joint>
+  <joint name="camera_color_joint" type="fixed">
+    <parent link="camera_link"/>
+    <child link="camera_color_frame"/>
+    <origin xyz="0 0.015 0" rpy="0 0 0"/>
+  </joint>
+  <joint name="camera_color_optical_joint" type="fixed">
+    <parent link="camera_color_frame"/>
+    <child link="camera_color_optical_frame"/>
     <origin xyz="0 0 0" rpy="-1.5707 0 -1.5707"/>
   </joint>

Commit message: added mapping tools and map convert

File: workspace/jig_description/urdf/gazebo_components.urdf.xacro (robot description, xacro)
@@ -2,9 +2,16 @@
 <robot xmlns:xacro="http://www.ros.org/wiki/xacro">
   <!-- ═══════════════════════════════════════════════════════════
-       GAZEBO SYSTEM PLUGINS
+       MODEL-LEVEL SYSTEMS
+       (Sensors/Imu systems could also live in the world SDF instead)
   ═══════════════════════════════════════════════════════════ -->
+  <!-- Gravity is a LINK property in SDF (a model-level <gravity> is ignored,
+       so the jig was really falling and the IMU read ~0 = free fall).
+       All fixed-joint children are lumped into base_link, so this covers the
+       whole jig. The IMU still reports world gravity (+9.81 m/s^2 up). -->
+  <gazebo reference="base_link">
+    <gravity>false</gravity>
+  </gazebo>
   <gazebo>
     <static>false</static>
-    <gravity>false</gravity>
     <plugin filename="libgz-sim-sensors-system.so"
             name="gz::sim::systems::Sensors">
@@ -12,47 +19,72 @@
     </plugin>
     <plugin filename="libgz-sim-imu-system.so"
-            name="gz::sim::systems::Imu">
+            name="gz::sim::systems::Imu"/>
+    <!-- Ground-truth odometry: for evaluation (evo) and for the
+         odom_source:=gt debug mode in mapping.launch.py -->
+    <plugin filename="gz-sim-odometry-publisher-system"
+            name="gz::sim::systems::OdometryPublisher">
+      <odom_frame>odom</odom_frame>
+      <robot_base_frame>base_link</robot_base_frame>
+      <odom_topic>/model/jig/odometry</odom_topic>
+      <tf_topic>/model/jig/odom_tf</tf_topic>
+      <odom_publish_frequency>50</odom_publish_frequency>
+      <dimensions>3</dimensions>
+    </plugin>
+    <!-- Body-frame velocity commands from jig_path_motion.py
+         (replaces set_pose teleporting so the IMU sees real motion) -->
+    <plugin filename="gz-sim-velocity-control-system"
+            name="gz::sim::systems::VelocityControl">
+      <topic>/model/jig/cmd_vel</topic>
     </plugin>
   </gazebo>
   <!-- ═══════════════════════════════════════════════════════════
-       LIDAR SENSOR (MID360)
+       LIDAR (Livox MID360 approximation)
+       Real: 360° H, -7°..+52° V, 0.1–40 m (@10% refl.), ≤2 cm, 10 Hz, ~200k pts/s
+       Note: Gazebo uses a repetitive scan pattern and no per-point time,
+       so keep deskewing disabled in sim.
   ═══════════════════════════════════════════════════════════ -->
   <gazebo reference="lidar_link">
     <sensor name="lidar_sensor" type="gpu_lidar">
+      <gz_frame_id>lidar_link</gz_frame_id>
       <always_on>true</always_on>
       <update_rate>10</update_rate>
       <topic>/scan</topic>
-      <visualize>true</visualize>
+      <visualize>false</visualize>
       <lidar>
         <scan>
           <horizontal>
-            <samples>420</samples>
+            <samples>600</samples>
             <resolution>1</resolution>
-            <min_angle>-3.1415</min_angle>
-            <max_angle>3.1415</max_angle>
+            <min_angle>-3.14159</min_angle>
+            <max_angle>3.13112</max_angle> <!-- π - one step: no duplicate column -->
           </horizontal>
           <vertical>
             <samples>40</samples>
             <resolution>1</resolution>
-            <min_angle>0</min_angle>
-            <max_angle>0.6109</max_angle>
+            <min_angle>-0.12217</min_angle> <!-- -7° -->
+            <max_angle>0.90757</max_angle>  <!-- +52° -->
           </vertical>
         </scan>
         <range>
-          <min>0.2</min>
-          <max>150</max>
-          <resolution>0.05</resolution>
+          <min>0.1</min>
+          <max>40.0</max>
+          <resolution>0.01</resolution>
         </range>
         <noise>
           <type>gaussian</type>
           <mean>0.0</mean>
-          <stddev>0.01</stddev>
+          <stddev>0.02</stddev>
         </noise>
       </lidar>
     </sensor>
-    <!-- ═══════════════════════════════════════════════════════
-         IMU SENSOR (built into MID360)
-    ═══════════════════════════════════════════════════════ -->
+  </gazebo>
+  <!-- ═══════════════════════════════════════════════════════════
+       IMU (MID360 built-in, ICM40609-class)
+       If you want the sim to mirror the real Spresense setup instead,
+       drop update_rate to ~22 Hz and tune noise to that IMU.
+  ═══════════════════════════════════════════════════════════ -->
+  <gazebo reference="imu_link">
     <sensor name="imu_sensor" type="imu">
+      <gz_frame_id>imu_link</gz_frame_id>
       <always_on>true</always_on>
       <update_rate>200</update_rate>
@@ -60,70 +92,39 @@
       <imu>
         <angular_velocity>
-          <x>
-            <noise type="gaussian">
-              <mean>0.0</mean>
-              <stddev>2e-4</stddev>
-              <bias_mean>0.0000075</bias_mean>
-              <bias_stddev>0.0000008</bias_stddev>
-            </noise>
-          </x>
-          <y>
-            <noise type="gaussian">
-              <mean>0.0</mean>
-              <stddev>2e-4</stddev>
-              <bias_mean>0.0000075</bias_mean>
-              <bias_stddev>0.0000008</bias_stddev>
-            </noise>
-          </y>
-          <z>
-            <noise type="gaussian">
-              <mean>0.0</mean>
-              <stddev>2e-4</stddev>
-              <bias_mean>0.0000075</bias_mean>
-              <bias_stddev>0.0000008</bias_stddev>
-            </noise>
-          </z>
+          <x><noise type="gaussian"><mean>0.0</mean><stddev>2e-4</stddev>
+            <bias_mean>7.5e-6</bias_mean><bias_stddev>8e-7</bias_stddev></noise></x>
+          <y><noise type="gaussian"><mean>0.0</mean><stddev>2e-4</stddev>
+            <bias_mean>7.5e-6</bias_mean><bias_stddev>8e-7</bias_stddev></noise></y>
+          <z><noise type="gaussian"><mean>0.0</mean><stddev>2e-4</stddev>
+            <bias_mean>7.5e-6</bias_mean><bias_stddev>8e-7</bias_stddev></noise></z>
         </angular_velocity>
         <linear_acceleration>
-          <x>
-            <noise type="gaussian">
-              <mean>0.0</mean>
-              <stddev>1.7e-2</stddev>
-              <bias_mean>0.1</bias_mean>
-              <bias_stddev>0.001</bias_stddev>
-            </noise>
-          </x>
-          <y>
-            <noise type="gaussian">
-              <mean>0.0</mean>
-              <stddev>1.7e-2</stddev>
-              <bias_mean>0.1</bias_mean>
-              <bias_stddev>0.001</bias_stddev>
-            </noise>
-          </y>
-          <z>
-            <noise type="gaussian">
-              <mean>0.0</mean>
-              <stddev>1.7e-2</stddev>
-              <bias_mean>0.1</bias_mean>
-              <bias_stddev>0.001</bias_stddev>
-            </noise>
-          </z>
+          <x><noise type="gaussian"><mean>0.0</mean><stddev>1.7e-2</stddev>
+            <bias_mean>0.01</bias_mean><bias_stddev>0.001</bias_stddev></noise></x>
+          <y><noise type="gaussian"><mean>0.0</mean><stddev>1.7e-2</stddev>
+            <bias_mean>0.01</bias_mean><bias_stddev>0.001</bias_stddev></noise></y>
+          <z><noise type="gaussian"><mean>0.0</mean><stddev>1.7e-2</stddev>
+            <bias_mean>0.01</bias_mean><bias_stddev>0.001</bias_stddev></noise></z>
         </linear_acceleration>
       </imu>
-      <plugin filename="libgz-sim-imu-system.so"
-              name="gz::sim::systems::Imu">
-      </plugin>
+      <!-- no <plugin> here: the Imu system is loaded once at model level -->
     </sensor>
   </gazebo>
-   <!-- ═══════════════════════════════════════════════════════════
-       REALSENSE D435 — RGB CAMERA
+  <!-- ═══════════════════════════════════════════════════════════
+       REALSENSE D435 — single RGB-D sensor (depth aligned to color,
+       same as the real driver with align_depth.enable:=true)
+       Publishes: /camera/image, /camera/depth_image,
+                  /camera/points, /camera/camera_info
   ═══════════════════════════════════════════════════════════ -->
   <gazebo reference="camera_color_frame">
-    <sensor name="rgb_camera" type="camera">
+    <sensor name="rgbd_camera" type="rgbd_camera">
+      <!-- Images must be stamped in the optical frame (z forward).
+           Its /camera/points output is x-forward data and is NOT bridged;
+           the cloud comes from the depth_cloud sensor below instead. -->
+      <gz_frame_id>camera_color_optical_frame</gz_frame_id>
       <always_on>true</always_on>
-      <update_rate>30</update_rate>
-      <topic>/camera/color/image_raw</topic>
-      <visualize>true</visualize>
+      <update_rate>15</update_rate>
+      <topic>/camera</topic>
+      <visualize>false</visualize>
       <camera>
         <horizontal_fov>1.2112</horizontal_fov>
@@ -134,6 +135,6 @@
         </image>
         <clip>
-          <near>0.1</near>
-          <far>100</far>
+          <near>0.2</near>
+          <far>10.0</far>
         </clip>
         <noise>
@@ -146,14 +147,22 @@
   </gazebo>
   <!-- ═══════════════════════════════════════════════════════════
-       REALSENSE D435 — DEPTH CAMERA
+       REALSENSE D435 — POINT CLOUD
+       Gazebo writes cloud XYZ in the link convention (x fwd, y left, z up),
+       so this sensor is stamped with camera_color_frame (same convention)
+       instead of the optical frame. Same pose, FOV and resolution as the
+       RGB-D sensor above, so the cloud is spatially aligned with the image
+       (organized 640x480: point (u,v) <-> pixel (u,v)). TF handles the
+       camera_color_frame -> camera_color_optical_frame rotation.
+       Publishes: /camera/cloud (depth, unused), /camera/cloud/points
   ═══════════════════════════════════════════════════════════ -->
-  <gazebo reference="camera_depth_frame">
-    <sensor name="depth_camera" type="depth_camera">
+  <gazebo reference="camera_color_frame">
+    <sensor name="depth_cloud" type="depth_camera">
+      <gz_frame_id>camera_color_frame</gz_frame_id>
       <always_on>true</always_on>
-      <update_rate>30</update_rate>
-      <topic>/camera/depth/image_rect_raw</topic>
-      <visualize>true</visualize>
+      <update_rate>15</update_rate>
+      <topic>/camera/cloud</topic>
+      <visualize>false</visualize>
       <camera>
-        <horizontal_fov>1.4835</horizontal_fov>
+        <horizontal_fov>1.2112</horizontal_fov>
         <image>
           <width>640</width>
@@ -162,5 +171,5 @@
         </image>
         <clip>
-          <near>0.1</near>
+          <near>0.2</near>
           <far>10.0</far>
         </clip>
@@ -168,8 +177,8 @@
           <type>gaussian</type>
           <mean>0.0</mean>
-          <stddev>0.01</stddev>
+          <stddev>0.007</stddev>
         </noise>
       </camera>
     </sensor>
   </gazebo>
-  </robot>
+</robot>

File: workspace/jig_description/urdf/lidar.urdf.xacro (robot description, xacro)
@@ -2,10 +2,14 @@
 <robot xmlns:xacro="http://www.ros.org/wiki/xacro">
   <!-- ═══════════════════════════════════════════════════════════
-       LIDAR PARAMETERS
+       LIDAR PARAMETERS  (single source of truth for the lidar pose)
   ═══════════════════════════════════════════════════════════ -->
-  <xacro:property name="lidar_xyz"         value="0.025 -0.005 0.035"/>
-  <xacro:property name="lidar_rpy"         value="0 1.57 0"/>
+  <xacro:property name="lidar_xyz" value="0.025 -0.005 0.035"/>
+  <xacro:property name="lidar_rpy" value="0 ${pi/2} 0"/>
+  <!-- MID360 internal IMU position in the lidar frame.
+       From FAST-LIO mid360.yaml (extrinsic_T = -0.011 -0.02329 0.04412 is
+       lidar-in-IMU, so IMU-in-lidar is the negation). Verify vs. Livox datasheet. -->
+  <xacro:property name="imu_in_lidar_xyz" value="0.011 0.02329 -0.04412"/>
   <!-- ═══════════════════════════════════════════════════════════
-       LIDAR LINK (MID360 with built-in IMU)
+       LIDAR LINK (MID360)
   ═══════════════════════════════════════════════════════════ -->
   <link name="lidar_link">
@@ -20,21 +24,19 @@
       </material>
     </visual>
+    <!-- Simple primitive collision: cheaper than the STL and avoids
+         self-hits from a detailed mesh -->
     <collision>
       <origin xyz="0 0 0" rpy="0 0 0"/>
       <geometry>
-        <mesh filename="package://jig_description/meshes/mid360.stl"
-              scale="0.001 0.001 0.001"/>
+        <cylinder radius="0.033" length="0.06"/>
       </geometry>
     </collision>
     <inertial>
       <origin xyz="0 0 0" rpy="0 0 0"/>
-      <mass value="0.3"/>
-      <inertia ixx="0.001" ixy="0" ixz="0"
-               iyy="0.001" iyz="0" izz="0.001"/>
+      <mass value="0.265"/>
+      <inertia ixx="0.0001" ixy="0" ixz="0"
+               iyy="0.0001" iyz="0" izz="0.0001"/>
     </inertial>
   </link>
-  <!-- ═══════════════════════════════════════════════════════════
-       LIDAR JOINT
-  ═══════════════════════════════════════════════════════════ -->
   <joint name="base_to_lidar" type="fixed">
     <parent link="base_link"/>
@@ -42,3 +44,12 @@
     <origin xyz="${lidar_xyz}" rpy="${lidar_rpy}"/>
   </joint>
+  <!-- ═══════════════════════════════════════════════════════════
+       IMU LINK (MID360 built-in IMU)
+  ═══════════════════════════════════════════════════════════ -->
+  <link name="imu_link"/>
+  <joint name="lidar_to_imu" type="fixed">
+    <parent link="lidar_link"/>
+    <child link="imu_link"/>
+    <origin xyz="${imu_in_lidar_xyz}" rpy="0 0 0"/>
+  </joint>
 </robot>
